File: AdderBreakoutV2.kicad_pcb (KiCad board)
At the start: 2 copper layers, 204 x 75.2 mm, 56 parts, among them J1 USB_B_Micro, SW1 SW_DIP_x08, SW2 SW_DIP_x08, U1 74LS83, U2 74LS83

Commit message: Add measurements
Parts:
- moved REF** 2.50 mm to (66.8, 136.5)
Other:
- board text added: "https://github.com/UARTman/BinAddBreakoutBoard"
Changed lines of the file:
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@@
   (general
     (thickness 1.6)
-    (drawings 47)
+    (drawings 50)
     (tracks 308)
     (zones 0)
@@
       (outputformat 1)
       (mirror false)
-      (drillshape 1)
+      (drillshape 0)
       (scaleselection 1)
-      (outputdirectory ""))
+      (outputdirectory "gerber"))
   )
   (net 0 "")
@@
   )
   (module Symbol:OSHW-Logo_11.4x12mm_SilkScreen (layer F.Cu)
-    (at 66.75 134)
+    (at 66.75 136.5)
     (descr "Open Source Hardware Logo")
     (tags "Logo OSHW")
@@
     )
   )
+  (dimension 75.25 (width 0.15) (layer Dwgs.User)
+    (gr_text "75.250 mm" (at 238.05 154.875 90) (layer Dwgs.User)
+      (effects (font (size 1 1) (thickness 0.15)))
+    )
+    (feature1 (pts (xy 235 117.25) (xy 237.336421 117.25)))
+    (feature2 (pts (xy 235 192.5) (xy 237.336421 192.5)))
+    (crossbar (pts (xy 236.75 192.5) (xy 236.75 117.25)))
+    (arrow1a (pts (xy 236.75 117.25) (xy 237.336421 118.376504)))
+    (arrow1b (pts (xy 236.75 117.25) (xy 236.163579 118.376504)))
+    (arrow2a (pts (xy 236.75 192.5) (xy 237.336421 191.373496)))
+    (arrow2b (pts (xy 236.75 192.5) (xy 236.163579 191.373496)))
+  )
+  (dimension 204.000153 (width 0.15) (layer Dwgs.User)
+    (gr_text "204.000 mm" (at 132.994126 197.168559 359.9297846) (layer Dwgs.User)
+      (effects (font (size 1 1) (thickness 0.15)))
+    )
+    (feature1 (pts (xy 235 192.5) (xy 234.995 196.579981)))
+    (feature2 (pts (xy 31 192.25) (xy 30.995 196.329981)))
+    (crossbar (pts (xy 30.995719 195.74356) (xy 234.995719 195.99356)))
+    (arrow1a (pts (xy 234.995719 195.99356) (xy 233.868497 196.5786)))
+    (arrow1b (pts (xy 234.995719 195.99356) (xy 233.869935 195.405759)))
+    (arrow2a (pts (xy 30.995719 195.74356) (xy 32.121503 196.331361)))
+    (arrow2b (pts (xy 30.995719 195.74356) (xy 32.122941 195.15852)))
+  )
+  (gr_text https://github.com/UARTman/BinAddBreakoutBoard (at 81 128) (layer F.SilkS)
+    (effects (font (size 1 1) (thickness 0.15)))
+  )
   (gr_text "Copyright (C) Gusev Anton, 2021" (at 73.75 125.5) (layer F.SilkS)
